File: input shift register.kicad_block/input shift register.kicad_sch (KiCad schematic)
At the start: 10 parts, among them U1 74HC165

Commit message: layout tweaks, added frame and label aroundm, figured device-level blocks could be labeled for clarity.
Parts:
- removed C1: 0,1uF, Capacitor_THT:C_Disc_D7.0mm_W2.5mm_P5.00mm, symbol Device:C_Small
- removed R1, R2, R3, R4, R5, R6, R7, R8: R10k, Resistor_THT:R_Axial_DIN0309_L9.0mm_D3.2mm_P12.70mm_Horizontal, symbol Device:R
- removed U1: 74HC165, Package_DIP:DIP-16_W7.62mm_Socket_LongPads, symbol 74xx:74HC165
- added C4: 0,1uF, Capacitor_THT:C_Disc_D7.0mm_W2.5mm_P5.00mm, symbol Device:C_Small
- added R19, R20, R21, R22, R23, R24, R25, R26: 10k, Resistor_THT:R_Axial_DIN0309_L9.0mm_D3.2mm_P12.70mm_Horizontal, symbol Device:R
- added U3: 74HC165, Package_DIP:DIP-16_W7.62mm_Socket_LongPads, symbol 74xx:74HC165
Connections:
- net GND: now also C4.2, U3.10 (DS), U3.15 (~{CE}), U3.8 (GND)
- net IS_CLOCK: now also U3.2 (CP)
- net IS_DATA: now also U3.9 (Q7)
- net IS_LATCH: now also U3.1 (~{PL})
- net VCC: now also C4.1, R19.1, R20.1, R21.1, R22.1, R23.1, R24.1, R25.1, R26.1, U3.16 (VCC)
- new net IS_SWITCH1: R19.2, U3.11 (D0)
- new net IS_SWITCH2: R20.2, U3.12 (D1)
- new net IS_SWITCH3: R21.2, U3.13 (D2)
- new net IS_SWITCH4: R22.2, U3.14 (D3)
- new net IS_SWITCH5: R23.2, U3.3 (D4)
- new net IS_SWITCH6: R24.2, U3.4 (D5)
- new net IS_SWITCH7: R25.2, U3.5 (D6)
- new net IS_SWITCH8: R26.2, U3.6 (D7)
Other:
- note added: "switches connect to input shifter the same as to microcontroller pins."
- note removed: "input shifter switches connect to GND like regular switches."
